Commit message: 一通りsdfをurdfに変更。動くようにはなった

File: nhk2023_simulator/launch/worlds/models/imu.urdf.xacro (robot description, xacro)
@@ -8,5 +8,21 @@
             <origin xyz="${xyz}" rpy="0 0 0"/>
         </joint>
-        <link name="${prefix}_link"/>
+        <link name="${prefix}_link">
+            <visual>
+                <geometry>
+                    <box size="0.1 0.1 0.1" />
+                </geometry>
+            </visual>
+            <collision>
+                <geometry>
+                    <box size="0.1 0.1 0.1" />
+                </geometry>
+            </collision>
+            <inertial>
+                <origin xyz="0 0 0" rpy="0 0 0" />
+                <mass value="0.1" />
+                <inertia ixx="0.0001" ixy="0" ixz="0" iyx="0" iyy="0.0001" iyz="0" izx="0" izy="0" izz="0.0001" />
+            </inertial>
+        </link>
         <gazebo reference="${prefix}_link">
             <gravity>true</gravity>
@@ -15,14 +31,5 @@
                 <update_rate>100</update_rate>
                 <visualize>true</visualize>
-                <topic>data</topic>
-                <plugin filename="libgazebo_ros_imu_sensor.so" name="imu_plugin">
-                    <topicName>${prefix}</topicName>                    <!--${prefix}/data-->
-                    <bodyName>${prefix}_link</bodyName>
-                    <updateRateHZ>30.0</updateRateHZ>
-                    <gaussianNoise>0.0</gaussianNoise>
-                    <xyzOffset>0 0 0</xyzOffset>
-                    <rpyOffset>0 0 0</rpyOffset>
-                    <frameName>${prefix}_link</frameName>
-                </plugin>
+                <topic>imu</topic>
                 <pose>0 0 0 0 0 0</pose>
             </sensor>

File: nhk2023_simulator/launch/worlds/models/lidar.urdf.xacro (robot description, xacro)
@@ -24,9 +24,9 @@
         <gazebo reference="${prefix}_link">
             <material>Gazebo/Red</material>
-            <sensor type="ray" name="${prefix}">
+            <sensor type="gpu_lidar" name="${prefix}">
                 <pose>0 0 0 0 0 0</pose>
                 <visualize>false</visualize>
                 <update_rate>10</update_rate>
-                <ray>
+                <lidar>
                     <scan>
                         <horizontal>
@@ -47,10 +47,8 @@
                         <stddev>0.01</stddev>
                     </noise>
-                </ray>
-                <plugin name="gazebo_ros_lidar_controller" filename="libgazebo_ros_laser.so">
-                    <topicName>/scan</topicName>
-                    <frameName>${prefix}_link</frameName>
-                </plugin>
+                </lidar>
             </sensor>
+            <plugin filename="libignition-gazebo-imu-system.so" name="ignition::gazebo::systems::Imu">
+            </plugin>
         </gazebo>
     </xacro:macro>

File: nhk2023_simulator/launch/worlds/models/simple_odom_robot.urdf.xacro (robot description, xacro)
@@ -2,6 +2,6 @@
 <robot name="odm_robot"
     xmlns:xacro="http://ros.org/wiki/xacro">
-    <xacro:include filename="$(find nhk2023_simulator)/urdf/lidar.urdf.xacro" />
-    <xacro:include filename="$(find nhk2023_simulator)/urdf/imu.urdf.xacro" />
+    <xacro:include filename="$(cwd)/lidar.urdf.xacro" />
+    <xacro:include filename="$(cwd)/imu.urdf.xacro" />
     <xacro:property name="PI" value="3.1415926535897931"/>
     <xacro:property name="b_m" value="20.0"/>
@@ -11,5 +11,4 @@
     <xacro:property name="b_h" value="0.1"/>
     <xacro:property name="b_d" value="0.60"/>
-    <xacro:property name="lidar_w" value="0.64"/>
     <material name="red">
         <color rgba="0.2 0 0 1"/>
@@ -60,6 +59,6 @@
     <material>Gazebo/Red</material>
   </gazebo> -->
-    <xacro:laser_macro prefix="lidar1" parent="base_link" xyz="${lidar_w/2} -${lidar_w/2} 0.04" rpy="0 0 -${PI/4}" />
-    <xacro:laser_macro prefix="lidar2" parent="base_link" xyz="-${lidar_w/2} ${lidar_w/2} 0.04" rpy="0 0 ${3*PI/4}" />
+    <xacro:laser_macro prefix="lidar" parent="base_link" xyz="0 ${b_w/2} 0.04" rpy="0 0 0" />
+    <!-- <xacro:laser_macro prefix="lidar2" parent="base_link" xyz="-${lidar_w/2} ${lidar_w/2} 0.04" rpy="0 0 ${3*PI/4}" /> -->
     <xacro:imu_macro prefix="imu" parent="base_link" xyz="0.0 0 0.10" />
     <gazebo>

Commit message: swerveモデルの追加

File: nhk2023_simulator/launch/worlds/models/imu.urdf.xacro (robot description, xacro)
@@ -25,14 +25,11 @@
             </inertial>
         </link>
-        <gazebo reference="${prefix}_link">
-            <gravity>true</gravity>
-            <sensor name="imu_sensor" type="imu">
-                <always_on>true</always_on>
-                <update_rate>100</update_rate>
-                <visualize>true</visualize>
-                <topic>imu</topic>
-                <pose>0 0 0 0 0 0</pose>
-            </sensor>
-        </gazebo>
+        <sensor name="imu_sensor" type="imu">
+            <always_on>true</always_on>
+            <update_rate>100</update_rate>
+            <visualize>true</visualize>
+            <topic>imu</topic>
+            <pose>0 0 0 0 0 0</pose>
+        </sensor>
     </xacro:macro>
 </robot>

File: nhk2023_simulator/launch/worlds/models/lidar.urdf.xacro (robot description, xacro)
@@ -22,34 +22,31 @@
             </collision>
         </link>
-        <gazebo reference="${prefix}_link">
-            <material>Gazebo/Red</material>
-            <sensor type="gpu_lidar" name="${prefix}">
-                <pose>0 0 0 0 0 0</pose>
-                <visualize>false</visualize>
-                <update_rate>10</update_rate>
-                <lidar>
-                    <scan>
-                        <horizontal>
-                            <samples>400</samples>
-                            <resolution>1</resolution>
-                            <min_angle>${radians(-180)}</min_angle>
-                            <max_angle>${radians(180)}</max_angle>
-                        </horizontal>
-                    </scan>
-                    <range>
-                        <min>0.10</min>
-                        <max>20.0</max>
-                        <resolution>0.01</resolution>
-                    </range>
-                    <noise>
-                        <type>gaussian</type>
-                        <mean>0.0</mean>
-                        <stddev>0.01</stddev>
-                    </noise>
-                </lidar>
-            </sensor>
-            <plugin filename="libignition-gazebo-imu-system.so" name="ignition::gazebo::systems::Imu">
-            </plugin>
-        </gazebo>
+        <sensor type="gpu_lidar" name="${prefix}">
+            <pose>0 0 0 0 0 0</pose>
+            <visualize>false</visualize>
+            <update_rate>10</update_rate>
+            <lidar>
+                <scan>
+                    <horizontal>
+                        <samples>400</samples>
+                        <resolution>1</resolution>
+                        <min_angle>${radians(-180)}</min_angle>
+                        <max_angle>${radians(180)}</max_angle>
+                    </horizontal>
+                </scan>
+                <range>
+                    <min>0.10</min>
+                    <max>20.0</max>
+                    <resolution>0.01</resolution>
+                </range>
+                <noise>
+                    <type>gaussian</type>
+                    <mean>0.0</mean>
+                    <stddev>0.01</stddev>
+                </noise>
+            </lidar>
+        </sensor>
+        <plugin filename="libignition-gazebo-imu-system.so" name="ignition::gazebo::systems::Imu">
+        </plugin>
     </xacro:macro>
 </robot>

File: nhk2023_simulator/launch/worlds/models/simple_odom_robot.urdf.xacro (robot description, xacro)
@@ -1,4 +1,4 @@
 <?xml version="1.0"?>
-<robot name="odm_robot"
+<robot name="er"
     xmlns:xacro="http://ros.org/wiki/xacro">
     <xacro:include filename="$(cwd)/lidar.urdf.xacro" />
@@ -62,7 +62,5 @@
     <!-- <xacro:laser_macro prefix="lidar2" parent="base_link" xyz="-${lidar_w/2} ${lidar_w/2} 0.04" rpy="0 0 ${3*PI/4}" /> -->
     <xacro:imu_macro prefix="imu" parent="base_link" xyz="0.0 0 0.10" />
-    <gazebo>
-        <plugin name="ignition::gazebo::systems::VelocityControl" filename="ignition-gazebo-velocity-control-system">
-        </plugin>
-    </gazebo>
+    <plugin name="ignition::gazebo::systems::VelocityControl" filename="ignition-gazebo-velocity-control-system">
+    </plugin>
 </robot>

File: nhk2023_simulator/launch/worlds/models/swerve_body.urdf.xacro (robot description, xacro)
@@ -1,12 +1,6 @@
 <?xml version="1.0" ?>
-<robot name="body"
+<model name="body"
     xmlns:xacro="http://ros.org/wiki/xacro">
-    <link name="base_footprint" />
     <link name="base_link" />
-    <joint name="base_joint" type="fixed">
-        <parent link="base_footprint" />
-        <child link="base_link" />
-        <origin xyz="0 0 0.01" rpy="0 0 0" />
-    </joint>
     <xacro:property name="b_m" value="5.58"/>
     <xacro:property name="b_m2" value="${b_m/12}"/>
@@ -32,8 +26,8 @@
         </inertial>
     </link>
-    <joint name="body_joint" type="fixed">
-        <parent link="base_footprint" />
+    <joint name="base_body_joint" type="fixed">
+        <parent link="base_link" />
         <child link="body" />
         <origin xyz="0 0 0.195" rpy="0 0 0" />
     </joint>
-</robot>
+</model>

File: nhk2023_simulator/launch/worlds/models/swerve_robot.urdf.xacro (robot description, xacro)
@@ -1,25 +1,14 @@
 <?xml version="1.0" ?>
-<robot name="simple_swerve"
+<robot name="rr_swerve"
     xmlns:xacro="http://ros.org/wiki/xacro">
-    <xacro:include filename="$(find nhk2023_simulator)/urdf/swerve_body.urdf.xacro" />
-    <xacro:include filename="$(find nhk2023_simulator)/urdf/swerve_wheel.urdf.xacro" />
-    <xacro:include filename="$(find nhk2023_simulator)/urdf/lidar.urdf.xacro" />
-    <xacro:include filename="$(find nhk2023_simulator)/urdf/imu.urdf.xacro" />
-    <xacro:include filename="$(find nhk2023_simulator)/urdf/_d435.urdf.xacro" />
-    <gazebo>
-        <plugin name="gazebo_ros_control" filename="libgazebo_ros_control.so">
-            <robotNamespace>/simple_swerve</robotNamespace>
-            <robotSimType>gazebo_ros_control/DefaultRobotHWSim</robotSimType>
-            <legacyModeNS>true</legacyModeNS>
-        </plugin>
-    </gazebo>
-    <xacro:wheel rl="rf" parent="base_footprint" />
-    <xacro:wheel rl="lf" parent="base_footprint" />
-    <xacro:wheel rl="rb" parent="base_footprint" />
-    <xacro:wheel rl="lb" parent="base_footprint" />
-    <xacro:laser_macro prefix="rplidar" parent="base_footprint" xyz="0.205 0 0.04" />
-    <xacro:imu_macro prefix="imu" parent="base_footprint" xyz="0.0 0 0.10" />
-    <sensor_d435 parent="rplidar_link">
-        <origin xyz="0.0 0.0 0.3" rpy="0 0.1745 0"/>
-    </sensor_d435>
+    <xacro:include filename="$(find nhk2023_simulator)/launch/worlds/models/swerve_body.urdf.xacro" />
+    <xacro:include filename="$(find nhk2023_simulator)/launch/worlds/models/swerve_wheel.urdf.xacro" />
+    <xacro:include filename="$(find nhk2023_simulator)/launch/worlds/models/lidar.urdf.xacro" />
+    <xacro:include filename="$(find nhk2023_simulator)/launch/worlds/models/imu.urdf.xacro" />
+    <xacro:wheel rl="rf" parent="base_link" />
+    <xacro:wheel rl="lf" parent="base_link" />
+    <xacro:wheel rl="rb" parent="base_link" />
+    <xacro:wheel rl="lb" parent="base_link" />
+    <xacro:laser_macro prefix="rplidar" parent="base_link" xyz="0.205 0 0.04" rpy="0 0 0"/>
+    <xacro:imu_macro prefix="imu" parent="base_link" xyz="0.0 0 0.10" />
 </robot>

File: nhk2023_simulator/launch/worlds/models/swerve_wheel.urdf.xacro (robot description, xacro)
@@ -1,4 +1,4 @@
 <?xml version="1.0" ?>
-<robot name="wheel"
+<model name="wheel"
     xmlns:xacro="http://ros.org/wiki/xacro">
     <xacro:property name="PI" value="3.1415926535897931"/>
@@ -40,4 +40,15 @@
                     <cylinder radius="${wheel_radius}" length="${wheel_height}" />
                 </geometry>
+                <surface>
+                    <friction>
+                        <ode>
+                            <mu>1</mu>
+                            <mu2>1</mu2>
+                            <slip1>0.035</slip1>
+                            <slip2>0</slip2>
+                            <fdir1>0 0 1</fdir1>
+                        </ode>
+                    </friction>
+                </surface>
             </collision>
             <inertial>
@@ -79,30 +90,8 @@
             <dynamics damping="0.1"/>
         </joint>
-        <gazebo reference="wheel_${rl}">
-            <material>Gazebo/Black</material>
-            <mu1 value="3.0" />
-            <!--friction-->
-            <mu2 value="3.0" />
-        </gazebo>
-        <transmission name="wheel_${rl}_trans" type="SimpleTransmission">
-            <type>transmission_interface/SimpleTransmission</type>
-            <actuator name="wheel_${rl}_motor">
-                <hardwareInterface>hardware_interface/EffortJointInterface</hardwareInterface>
-                <mechanicalReduction>1</mechanicalReduction>
-            </actuator>
-            <joint name="wheel_${rl}_joint">
-                <hardwareInterface>hardware_interface/EffortJointInterface</hardwareInterface>
-            </joint>
-        </transmission>
-        <transmission name="wheel_${rl}_angular_trans" type="SimpleTransmission">
-            <type>transmission_interface/SimpleTransmission</type>
-            <actuator name="wheel_${rl}_angular_motor">
-                <hardwareInterface>hardware_interface/EffortJointInterface</hardwareInterface>
-                <mechanicalReduction>1</mechanicalReduction>
-            </actuator>
-            <joint name="wheel_${rl}_angular_joint">
-                <hardwareInterface>hardware_interface/EffortJointInterface</hardwareInterface>
-            </joint>
-        </transmission>
+        <plugin filename="gz-sim-joint-controller-system" name="gz::sim::systems::JointController">
+            <joint_name>wheel_${rl}_angular_joint</joint_name>
+            <initial_velocity>5.0</initial_velocity>
+        </plugin>
     </xacro:macro>
-</robot>
+</model>

Commit message: urdfからsdfの変換の際に情報がすべて抜け落ちる、理由は不マイ

File: nhk2023_simulator/launch/worlds/models/imu.urdf.xacro (robot description, xacro)
@@ -24,12 +24,12 @@
                 <inertia ixx="0.0001" ixy="0" ixz="0" iyx="0" iyy="0.0001" iyz="0" izx="0" izy="0" izz="0.0001" />
             </inertial>
+            <sensor name="imu_sensor" type="imu">
+                <always_on>true</always_on>
+                <update_rate>100</update_rate>
+                <visualize>true</visualize>
+                <topic>imu</topic>
+                <pose>0 0 0 0 0 0</pose>
+            </sensor>
         </link>
-        <sensor name="imu_sensor" type="imu">
-            <always_on>true</always_on>
-            <update_rate>100</update_rate>
-            <visualize>true</visualize>
-            <topic>imu</topic>
-            <pose>0 0 0 0 0 0</pose>
-        </sensor>
     </xacro:macro>
 </robot>

File: nhk2023_simulator/launch/worlds/models/lidar.urdf.xacro (robot description, xacro)
@@ -13,5 +13,4 @@
                     <cylinder radius="0.02" length="0.06" />
                 </geometry>
-                <material name="red" />
             </visual>
             <collision>
@@ -21,30 +20,30 @@
                 </geometry>
             </collision>
+            <sensor type="gpu_lidar" name="${prefix}">
+                <pose>0 0 0 0 0 0</pose>
+                <visualize>false</visualize>
+                <update_rate>10</update_rate>
+                <lidar>
+                    <scan>
+                        <horizontal>
+                            <samples>400</samples>
+                            <resolution>1</resolution>
+                            <min_angle>${radians(-180)}</min_angle>
+                            <max_angle>${radians(180)}</max_angle>
+                        </horizontal>
+                    </scan>
+                    <range>
+                        <min>0.10</min>
+                        <max>20.0</max>
+                        <resolution>0.01</resolution>
+                    </range>
+                    <noise>
+                        <type>gaussian</type>
+                        <mean>0.0</mean>
+                        <stddev>0.01</stddev>
+                    </noise>
+                </lidar>
+            </sensor>
         </link>
-        <sensor type="gpu_lidar" name="${prefix}">
-            <pose>0 0 0 0 0 0</pose>
-            <visualize>false</visualize>
-            <update_rate>10</update_rate>
-            <lidar>
-                <scan>
-                    <horizontal>
-                        <samples>400</samples>
-                        <resolution>1</resolution>
-                        <min_angle>${radians(-180)}</min_angle>
-                        <max_angle>${radians(180)}</max_angle>
-                    </horizontal>
-                </scan>
-                <range>
-                    <min>0.10</min>
-                    <max>20.0</max>
-                    <resolution>0.01</resolution>
-                </range>
-                <noise>
-                    <type>gaussian</type>
-                    <mean>0.0</mean>
-                    <stddev>0.01</stddev>
-                </noise>
-            </lidar>
-        </sensor>
         <plugin filename="libignition-gazebo-imu-system.so" name="ignition::gazebo::systems::Imu">
         </plugin>

File: nhk2023_simulator/launch/worlds/models/swerve_body.urdf.xacro (robot description, xacro)
@@ -1,4 +1,4 @@
 <?xml version="1.0" ?>
-<model name="body"
+<robot name="body"
     xmlns:xacro="http://ros.org/wiki/xacro">
     <link name="base_link" />
@@ -31,3 +31,3 @@
         <origin xyz="0 0 0.195" rpy="0 0 0" />
     </joint>
-</model>
+</robot>

File: nhk2023_simulator/launch/worlds/models/swerve_wheel.urdf.xacro (robot description, xacro)
@@ -1,4 +1,4 @@
 <?xml version="1.0" ?>
-<model name="wheel"
+<robot name="wheel"
     xmlns:xacro="http://ros.org/wiki/xacro">
     <xacro:property name="PI" value="3.1415926535897931"/>
@@ -95,3 +95,3 @@
         </plugin>
     </xacro:macro>
-</model>
+</robot>
