Commit message: すごく微妙なところだけど一旦コミット、これねそもそもsdfへの変換が上手くいっていない…どうすりゃ

File: nhk2023_simulator/launch/worlds/models/imu.urdf.xacro (robot description, xacro)
@@ -3,8 +3,9 @@
     xmlns:xacro="http://ros.org/wiki/xacro">
     <xacro:macro name="imu_macro" params="parent prefix xyz">
-        <joint name="imu_joint" type="fixed">
+        <joint name="imu_joint" type="revolute">
             <parent link="${parent}"/>
             <child link="${prefix}_link"/>
             <origin xyz="${xyz}" rpy="0 0 0"/>
+            <limit lower="0" upper="0" effort="0" velocity="0"/>
         </joint>
         <link name="${prefix}_link">
@@ -24,4 +25,6 @@
                 <inertia ixx="0.0001" ixy="0" ixz="0" iyx="0" iyy="0.0001" iyz="0" izx="0" izy="0" izz="0.0001" />
             </inertial>
+        </link>
+        <gazebo>
             <sensor name="imu_sensor" type="imu">
                 <always_on>true</always_on>
@@ -31,5 +34,115 @@
                 <pose>0 0 0 0 0 0</pose>
             </sensor>
-        </link>
+            <plugin filename="ignition-gazebo-imu-system" name="ignition::gazebo::systems::Imu">
+                <imu_name>imu_sensor</imu_name>
+                <topic>imu</topic>
+                <frame_name>imu_link</frame_name>
+                <linear_acceleration>
+                    <x>
+                        <noise type="gaussian">
+                            <mean>0</mean>
+                            <stddev>0.0001</stddev>
+                            <bias_mean>0.0001</bias_mean>
+                            <bias_stddev>0.0001</bias_stddev>
+                            <dynamic_bias_stddev>0.0001</dynamic_bias_stddev>
+                            <dynamic_bias_correlation_time>1000.0</dynamic_bias_correlation_time>
+                            <precision>0.0001</precision>
+                        </noise>
+                    </x>
+                    <y>
+                        <noise type="gaussian">
+                            <mean>0</mean>
+                            <stddev>0.0001</stddev>
+                            <bias_mean>0.0001</bias_mean>
+                            <bias_stddev>0.0001</bias_stddev>
+                            <dynamic_bias_stddev>0.0001</dynamic_bias_stddev>
+                            <dynamic_bias_correlation_time>1000.0</dynamic_bias_correlation_time>
+                            <precision>0.0001</precision>
+                        </noise>
+                    </y>
+                    <z>
+                        <noise type="gaussian">
+                            <mean>0</mean>
+                            <stddev>0.0001</stddev>
+                            <bias_mean>0.0001</bias_mean>
+                            <bias_stddev>0.0001</bias_stddev>
+                            <dynamic_bias_stddev>0.0001</dynamic_bias_stddev>
+                            <dynamic_bias_correlation_time>1000.0</dynamic_bias_correlation_time>
+                            <precision>0.0001</precision>
+                        </noise>
+                    </z>
+                </linear_acceleration>
+                <angular_velocity>
+                    <x>
+                        <noise type="gaussian">
+                            <mean>0</mean>
+                            <stddev>0.0001</stddev>
+                            <bias_mean>0.0001</bias_mean>
+                            <bias_stddev>0.0001</bias_stddev>
+                            <dynamic_bias_stddev>0.0001</dynamic_bias_stddev>
+                            <dynamic_bias_correlation_time>1000.0</dynamic_bias_correlation_time>
+                            <precision>0.0001</precision>
+                        </noise>
+                    </x>
+                    <y>
+                        <noise type="gaussian">
+                            <mean>0</mean>
+                            <stddev>0.0001</stddev>
+                            <bias_mean>0.0001</bias_mean>
+                            <bias_stddev>0.0001</bias_stddev>
+                            <dynamic_bias_stddev>0.0001</dynamic_bias_stddev>
+                            <dynamic_bias_correlation_time>1000.0</dynamic_bias_correlation_time>
+                            <precision>0.0001</precision>
+                        </noise>
+                    </y>
+                    <z>
+                        <noise type="gaussian">
+                            <mean>0</mean>
+                            <stddev>0.0001</stddev>
+                            <bias_mean>0.0001</bias_mean>
+                            <bias_stddev>0.0001</bias_stddev>
+                            <dynamic_bias_stddev>0.0001</dynamic_bias_stddev>
+                            <dynamic_bias_correlation_time>1000.0</dynamic_bias_correlation_time>
+                            <precision>0.0001</precision>
+                        </noise>
+                    </z>
+                </angular_velocity>
+                <orientation>
+                    <x>
+                        <noise type="gaussian">
+                            <mean>0</mean>
+                            <stddev>0.0001</stddev>
+                            <bias_mean>0.0001</bias_mean>
+                            <bias_stddev>0.0001</bias_stddev>
+                            <dynamic_bias_stddev>0.0001</dynamic_bias_stddev>
+                            <dynamic_bias_correlation_time>1000.0</dynamic_bias_correlation_time>
+                            <precision>0.0001</precision>
+                        </noise>
+                    </x>
+                    <y>
+                        <noise type="gaussian">
+                            <mean>0</mean>
+                            <stddev>0.0001</stddev>
+                            <bias_mean>0.0001</bias_mean>
+                            <bias_stddev>0.0001</bias_stddev>
+                            <dynamic_bias_stddev>0.0001</dynamic_bias_stddev>
+                            <dynamic_bias_correlation_time>1000.0</dynamic_bias_correlation_time>
+                            <precision>0.0001</precision>
+                        </noise>
+                    </y>
+                    <z>
+                        <noise type="gaussian">
+                            <mean>0</mean>
+                            <stddev>0.0001</stddev>
+                            <bias_mean>0.0001</bias_mean>
+                            <bias_stddev>0.0001</bias_stddev>
+                            <dynamic_bias_stddev>0.0001</dynamic_bias_stddev>
+                            <dynamic_bias_correlation_time>1000.0</dynamic_bias_correlation_time>
+                            <precision>0.0001</precision>
+                        </noise>
+                    </z>
+                </orientation>
+            </plugin>
+        </gazebo>
     </xacro:macro>
 </robot>

File: nhk2023_simulator/launch/worlds/models/lidar.urdf.xacro (robot description, xacro)
@@ -1,9 +1,12 @@
+<?xml version="1.0" ?>
 <robot name="lidar"
     xmlns:xacro="http://ros.org/wiki/xacro">
     <xacro:macro name="laser_macro" params="parent prefix xyz rpy">
-        <joint name="${prefix}_joint" type="fixed">
+        <!-- <xacro:property name="radians" value="0.017453292519943295"/> -->
+        <joint name="${prefix}_joint" type="revolute">
             <parent link="${parent}"/>
             <child link="${prefix}_link"/>
             <origin xyz="${xyz}" rpy="${rpy}"/>
+            <limit lower="0" upper="0" effort="0" velocity="0"/>
         </joint>
         <link name="${prefix}_link">
@@ -20,4 +23,9 @@
                 </geometry>
             </collision>
+            <inertial>
+                <origin xyz="0 0 0" rpy="0 0 0" />
+                <mass value="0.2" />
+                <inertia ixx="0.0001" ixy="0" ixz="0" iyx="0" iyy="0.0001" iyz="0" izx="0" izy="0" izz="0.0001" />
+            </inertial>
             <sensor type="gpu_lidar" name="${prefix}">
                 <pose>0 0 0 0 0 0</pose>
@@ -29,6 +37,6 @@
                             <samples>400</samples>
                             <resolution>1</resolution>
-                            <min_angle>${radians(-180)}</min_angle>
-                            <max_angle>${radians(180)}</max_angle>
+                            <min_angle>-3.05433</min_angle>
+                            <max_angle>3.05433</max_angle>
                         </horizontal>
                     </scan>
@@ -46,6 +54,6 @@
             </sensor>
         </link>
-        <plugin filename="libignition-gazebo-imu-system.so" name="ignition::gazebo::systems::Imu">
-        </plugin>
+        <gazebo>
+        </gazebo>
     </xacro:macro>
 </robot>

File: nhk2023_simulator/launch/worlds/models/swerve_body.urdf.xacro (robot description, xacro)
@@ -2,6 +2,6 @@
 <robot name="body"
     xmlns:xacro="http://ros.org/wiki/xacro">
-    <link name="base_link" />
-    <xacro:property name="b_m" value="5.58"/>
+    <link name="base_link"/>
+    <xacro:property name="b_m" value="10"/>
     <xacro:property name="b_m2" value="${b_m/12}"/>
     <!--for calculation of inertia-->
@@ -30,4 +30,5 @@
         <child link="body" />
         <origin xyz="0 0 0.195" rpy="0 0 0" />
+        <!-- <limit lower="0" upper="0" effort="0" velocity="0" /> -->
     </joint>
 </robot>

File: nhk2023_simulator/launch/worlds/models/swerve_robot.urdf (robot description, URDF)
Before this commit: robot rr_swerve, 12 links, 11 joints
Links:
- removed link rplidar_link
- added link lidar_link, mass 0.2; collision cylinder length=0.06 radius=0.02; visual cylinder length=0.06 radius=0.02
- link body: mass 5.58 -> 10
Joints:
- removed joint rplidar_joint
- added joint lidar_joint: type revolute, parent base_link, child lidar_link, origin xyz=0.205 0 0.04 rpy=0 0 0, limit lower=0 upper=0 effort=0 velocity=0
- joint imu_joint: limit (none) -> lower=0 upper=0 effort=0 velocity=0; type fixed -> revolute

File: nhk2023_simulator/launch/worlds/models/swerve_robot.urdf.xacro (robot description, xacro)
@@ -10,5 +10,5 @@
     <xacro:wheel rl="rb" parent="base_link" />
     <xacro:wheel rl="lb" parent="base_link" />
-    <xacro:laser_macro prefix="rplidar" parent="base_link" xyz="0.205 0 0.04" rpy="0 0 0"/>
+    <xacro:laser_macro prefix="lidar" parent="base_link" xyz="0.205 0 0.04" rpy="0 0 0"/>
     <xacro:imu_macro prefix="imu" parent="base_link" xyz="0.0 0 0.10" />
 </robot>

File: nhk2023_simulator/launch/worlds/models/swerve_wheel.urdf.xacro (robot description, xacro)
@@ -90,8 +90,10 @@
             <dynamics damping="0.1"/>
         </joint>
-        <plugin filename="gz-sim-joint-controller-system" name="gz::sim::systems::JointController">
-            <joint_name>wheel_${rl}_angular_joint</joint_name>
-            <initial_velocity>5.0</initial_velocity>
-        </plugin>
+        <gazebo>
+            <plugin filename="ignition-gazebo-joint-controller-system" name="ignition::gazebo::systems::JointController">
+                <joint_name>wheel_${rl}_joint</joint_name>
+                <joint_name>wheel_${rl}_angular_joint</joint_name>
+            </plugin>
+        </gazebo>
     </xacro:macro>
 </robot>

Commit message: 作業環境変更

File: nhk2023_simulator/launch/worlds/models/imu.urdf.xacro (robot description, xacro)
@@ -25,6 +25,4 @@
                 <inertia ixx="0.0001" ixy="0" ixz="0" iyx="0" iyy="0.0001" iyz="0" izx="0" izy="0" izz="0.0001" />
             </inertial>
-        </link>
-        <gazebo>
             <sensor name="imu_sensor" type="imu">
                 <always_on>true</always_on>
@@ -34,114 +32,6 @@
                 <pose>0 0 0 0 0 0</pose>
             </sensor>
-            <plugin filename="ignition-gazebo-imu-system" name="ignition::gazebo::systems::Imu">
-                <imu_name>imu_sensor</imu_name>
-                <topic>imu</topic>
-                <frame_name>imu_link</frame_name>
-                <linear_acceleration>
-                    <x>
-                        <noise type="gaussian">
-                            <mean>0</mean>
-                            <stddev>0.0001</stddev>
-                            <bias_mean>0.0001</bias_mean>
-                            <bias_stddev>0.0001</bias_stddev>
-                            <dynamic_bias_stddev>0.0001</dynamic_bias_stddev>
-                            <dynamic_bias_correlation_time>1000.0</dynamic_bias_correlation_time>
-                            <precision>0.0001</precision>
-                        </noise>
-                    </x>
-                    <y>
-                        <noise type="gaussian">
-                            <mean>0</mean>
-                            <stddev>0.0001</stddev>
-                            <bias_mean>0.0001</bias_mean>
-                            <bias_stddev>0.0001</bias_stddev>
-                            <dynamic_bias_stddev>0.0001</dynamic_bias_stddev>
-                            <dynamic_bias_correlation_time>1000.0</dynamic_bias_correlation_time>
-                            <precision>0.0001</precision>
-                        </noise>
-                    </y>
-                    <z>
-                        <noise type="gaussian">
-                            <mean>0</mean>
-                            <stddev>0.0001</stddev>
-                            <bias_mean>0.0001</bias_mean>
-                            <bias_stddev>0.0001</bias_stddev>
-                            <dynamic_bias_stddev>0.0001</dynamic_bias_stddev>
-                            <dynamic_bias_correlation_time>1000.0</dynamic_bias_correlation_time>
-                            <precision>0.0001</precision>
-                        </noise>
-                    </z>
-                </linear_acceleration>
-                <angular_velocity>
-                    <x>
-                        <noise type="gaussian">
-                            <mean>0</mean>
-                            <stddev>0.0001</stddev>
-                            <bias_mean>0.0001</bias_mean>
-                            <bias_stddev>0.0001</bias_stddev>
-                            <dynamic_bias_stddev>0.0001</dynamic_bias_stddev>
-                            <dynamic_bias_correlation_time>1000.0</dynamic_bias_correlation_time>
-                            <precision>0.0001</precision>
-                        </noise>
-                    </x>
-                    <y>
-                        <noise type="gaussian">
-                            <mean>0</mean>
-                            <stddev>0.0001</stddev>
-                            <bias_mean>0.0001</bias_mean>
-                            <bias_stddev>0.0001</bias_stddev>
-                            <dynamic_bias_stddev>0.0001</dynamic_bias_stddev>
-                            <dynamic_bias_correlation_time>1000.0</dynamic_bias_correlation_time>
-                            <precision>0.0001</precision>
-                        </noise>
-                    </y>
-                    <z>
-                        <noise type="gaussian">
-                            <mean>0</mean>
-                            <stddev>0.0001</stddev>
-                            <bias_mean>0.0001</bias_mean>
-                            <bias_stddev>0.0001</bias_stddev>
-                            <dynamic_bias_stddev>0.0001</dynamic_bias_stddev>
-                            <dynamic_bias_correlation_time>1000.0</dynamic_bias_correlation_time>
-                            <precision>0.0001</precision>
-                        </noise>
-                    </z>
-                </angular_velocity>
-                <orientation>
-                    <x>
-                        <noise type="gaussian">
-                            <mean>0</mean>
-                            <stddev>0.0001</stddev>
-                            <bias_mean>0.0001</bias_mean>
-                            <bias_stddev>0.0001</bias_stddev>
-                            <dynamic_bias_stddev>0.0001</dynamic_bias_stddev>
-                            <dynamic_bias_correlation_time>1000.0</dynamic_bias_correlation_time>
-                            <precision>0.0001</precision>
-                        </noise>
-                    </x>
-                    <y>
-                        <noise type="gaussian">
-                            <mean>0</mean>
-                            <stddev>0.0001</stddev>
-                            <bias_mean>0.0001</bias_mean>
-                            <bias_stddev>0.0001</bias_stddev>
-                            <dynamic_bias_stddev>0.0001</dynamic_bias_stddev>
-                            <dynamic_bias_correlation_time>1000.0</dynamic_bias_correlation_time>
-                            <precision>0.0001</precision>
-                        </noise>
-                    </y>
-                    <z>
-                        <noise type="gaussian">
-                            <mean>0</mean>
-                            <stddev>0.0001</stddev>
-                            <bias_mean>0.0001</bias_mean>
-                            <bias_stddev>0.0001</bias_stddev>
-                            <dynamic_bias_stddev>0.0001</dynamic_bias_stddev>
-                            <dynamic_bias_correlation_time>1000.0</dynamic_bias_correlation_time>
-                            <precision>0.0001</precision>
-                        </noise>
-                    </z>
-                </orientation>
-            </plugin>
+        </link>
+        <gazebo>
         </gazebo>
     </xacro:macro>
