Commit message: シミュレーターに時間を取られていては何も生まないと気づいたのでこれで開発を打ち切ります

File: nhk2023_simulator/launch/worlds/models/swerve_body.urdf.xacro (robot description, xacro)
@@ -2,5 +2,21 @@
 <robot name="body"
     xmlns:xacro="http://ros.org/wiki/xacro">
-    <link name="base_link"/>
+    <link name="base_link">
+        <visual>
+            <geometry>
+                <box size="0.01 0.01 0.01" />
+            </geometry>
+        </visual>
+        <collision>
+            <geometry>
+                <box size="0.01 0.01 0.01" />
+            </geometry>
+        </collision>
+        <inertial>
+            <origin xyz="0 0 0" rpy="0 0 0" />
+            <mass value="0.1" />
+            <inertia ixx="0.0001" ixy="0" ixz="0" iyx="0" iyy="0.0001" iyz="0" izx="0" izy="0" izz="0.0001" />
+        </inertial>
+    </link>
     <xacro:property name="b_m" value="10"/>
     <xacro:property name="b_m2" value="${b_m/12}"/>
@@ -26,9 +42,9 @@
         </inertial>
     </link>
-    <joint name="base_body_joint" type="fixed">
+    <joint name="base_body_joint" type="revolute">
         <parent link="base_link" />
         <child link="body" />
         <origin xyz="0 0 0.195" rpy="0 0 0" />
-        <!-- <limit lower="0" upper="0" effort="0" velocity="0" /> -->
+        <limit lower="0" upper="0" effort="0" velocity="0" />
     </joint>
 </robot>

File: nhk2023_simulator/launch/worlds/models/swerve_robot.urdf (robot description, URDF)
Before this commit: robot rr_swerve, 12 links, 11 joints
Links:
- link base_link: mass None -> 0.1; geometry collision box size=0.01 0.01 0.01; visual box size=0.01 0.01 0.01
Joints:
- joint base_body_joint: limit (none) -> lower=0 upper=0 effort=0 velocity=0; type fixed -> revolute
