Commit message: とりあえずこみっつ

File: nhk2023_simulator/models/swerve_body.urdf.xacro (robot description, xacro)
@@ -1,50 +1,50 @@
 <?xml version="1.0" ?>
 <robot name="body"
-    xmlns:xacro="http://ros.org/wiki/xacro">
-    <link name="base_link">
-        <visual>
-            <geometry>
-                <box size="0.01 0.01 0.01" />
-            </geometry>
-        </visual>
-        <collision>
-            <geometry>
-                <box size="0.01 0.01 0.01" />
-            </geometry>
-        </collision>
-        <inertial>
-            <origin xyz="0 0 0" rpy="0 0 0" />
-            <mass value="0.1" />
-            <inertia ixx="0.0001" ixy="0" ixz="0" iyx="0" iyy="0.0001" iyz="0" izx="0" izy="0" izz="0.0001" />
-        </inertial>
-    </link>
-    <xacro:property name="b_m" value="10"/>
-    <xacro:property name="b_m2" value="${b_m/12}"/>
-    <!--for calculation of inertia-->
-    <xacro:property name="b_w" value="0.37"/>
-    <xacro:property name="b_h" value="0.37"/>
-    <xacro:property name="b_d" value="0.37"/>
-    <link name="body">
-        <visual>
-            <geometry>
-                <box size="${b_d} ${b_w} ${b_h}" />
-            </geometry>
-        </visual>
-        <collision>
-            <geometry>
-                <box size="${b_d*0.95} ${b_w*0.95} ${b_h*0.95}" />
-            </geometry>
-        </collision>
-        <inertial>
-            <origin xyz="0 0 0" rpy="0 0 0" />
-            <mass value="${b_m}" />
-            <inertia ixx="${b_m2*(b_h*b_h+b_w*b_w)}" ixy="0" ixz="0" iyx="0" iyy="${b_m2*(b_h*b_h+b_d*b_d)}" iyz="0" izx="0" izy="0" izz="${b_m2*(b_w*b_w+b_d*b_d)}" />
-        </inertial>
-    </link>
-    <joint name="base_body_joint" type="revolute">
-        <parent link="base_link" />
-        <child link="body" />
-        <origin xyz="0 0 0.195" rpy="0 0 0" />
-        <limit lower="0" upper="0" effort="0" velocity="0" />
-    </joint>
+  xmlns:xacro="http://ros.org/wiki/xacro">
+  <link name="base_link">
+    <visual>
+      <geometry>
+        <box size="0.01 0.01 0.01" />
+      </geometry>
+    </visual>
+    <collision>
+      <geometry>
+        <box size="0.01 0.01 0.01" />
+      </geometry>
+    </collision>
+    <inertial>
+      <origin xyz="0 0 0" rpy="0 0 0" />
+      <mass value="0.1" />
+      <inertia ixx="0.0001" ixy="0" ixz="0" iyx="0" iyy="0.0001" iyz="0" izx="0" izy="0" izz="0.0001" />
+    </inertial>
+  </link>
+  <xacro:property name="b_m" value="10"/>
+  <xacro:property name="b_m2" value="${b_m/12}"/>
+  <!--for calculation of inertia-->
+  <xacro:property name="b_w" value="0.37"/>
+  <xacro:property name="b_h" value="0.37"/>
+  <xacro:property name="b_d" value="0.37"/>
+  <link name="body">
+    <visual>
+      <geometry>
+        <box size="${b_d} ${b_w} ${b_h}" />
+      </geometry>
+    </visual>
+    <collision>
+      <geometry>
+        <box size="${b_d*0.95} ${b_w*0.95} ${b_h*0.95}" />
+      </geometry>
+    </collision>
+    <inertial>
+      <origin xyz="0 0 0" rpy="0 0 0" />
+      <mass value="${b_m}" />
+      <inertia ixx="${b_m2*(b_h*b_h+b_w*b_w)}" ixy="0" ixz="0" iyx="0" iyy="${b_m2*(b_h*b_h+b_d*b_d)}" iyz="0" izx="0" izy="0" izz="${b_m2*(b_w*b_w+b_d*b_d)}" />
+    </inertial>
+  </link>
+  <joint name="base_body_joint" type="revolute">
+    <parent link="base_link" />
+    <child link="body" />
+    <origin xyz="0 0 0.195" rpy="0 0 0" />
+    <limit lower="0" upper="0" effort="0" velocity="0" />
+  </joint>
 </robot>
