Commit message: うーん無理すぎ

File: nhk2023_simulator/models/rr/rr.urdf (robot description, URDF)
Before this commit: robot rr_swerve, 12 links, 11 joints
Links:
- link body: mass 10 -> 300

File: nhk2023_simulator/models/swerve_body.urdf.xacro (robot description, xacro)
@@ -19,5 +19,5 @@
     </inertial>
   </link>
-  <xacro:property name="b_m" value="10"/>
+  <xacro:property name="b_m" value="300"/>
   <xacro:property name="b_m2" value="${b_m/12}"/>
   <!--for calculation of inertia-->
